File: Drone/Drone/_autosave-Drone.kicad_sch (KiCad schematic)
At the start: 44 parts

Commit message: Schematic done
Parts:
- R?: value 5.6k -> 560
Changed lines of the file:
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@@
       (effects (font (size 1.27 1.27)) (justify left))
     )
-    (property "Value" "5.6k" (id 1) (at 50.8 107.315 90)
+    (property "Value" "560" (id 1) (at 50.8 107.315 90)
       (effects (font (size 1.27 1.27)) (justify left))
     )
@@
     )
     (path "/8405f1d0-5223-43ca-a0a0-545311a2ff9b"
-      (reference "R?") (unit 1) (value "5.6k") (footprint "")
+      (reference "R?") (unit 1) (value "560") (footprint "")
     )
     (path "/8e74bd62-30fd-4dc6-a6e9-8583d6626b7d"
